File: XL6009.kicad_pcb (KiCad board)
At the start: 2 copper layers, 29 x 44 mm, 20 parts, among them J1 Conn_01x02_Female, J2 Conn_01x03_Female, U1 XL6009

Commit message: Rev. A
Parts:
- turned C5 to 0 degrees
- turned C6 to 0 degrees
- turned C7 to 0 degrees
- turned C8 to 0 degrees
Routing:
- net Net-(C6-Pad2): track 25.8 -> 21.2 mm
- net Net-(C5-Pad1): track 14.9 -> 10.3 mm
- net GND: vias 43 -> 56
Other:
- board text added: "V-IN (3.7V)"
- board text removed: "Batt"

Commit message: initial
Other:
- net class Default removed
